File: 001-led/001-led.kicad_pcb (KiCad board)
At the start: 2 copper layers, 26.7 x 22.9 mm, 7 parts

Commit message: 001 again
Parts:
- removed REF** (x4): M2, MountingHole:MountingHole_2.2mm_M2
- BT1: value 9V -> Battery_Cell
- D1: footprint LED_SMD:LED_1206_3216Metric_Castellated -> LED_SMD:LED_0603_1608Metric
- R1: value 470 -> R; footprint Resistor_SMD:R_1206_3216Metric -> Resistor_SMD:R_0603_1608Metric
- moved R1 29.9 mm to (128.8, 122.6)
- moved D1 29.2 mm to (128.7, 125.1), turned to 0 degrees
- moved BT1 25.1 mm to (124.6, 122.6)
Connections:
- net Net-(BT1-Pad2) renamed GNDREF
Routing:
- net GNDREF: track 18.2 -> 0.00 mm, vias 1 -> 0
- net Net-(BT1-Pad1): track 9.45 -> 3.40 mm
- net Net-(D1-Pad2): track 7.36 -> 2.55 mm
- added copper zone on F.Cu, net GNDREF
- removed copper zone on B.Cu, net GNDREF
- removed copper zone on F.Cu, net Net-(BT1-Pad1)
Other:
- board size 26.7 x 22.9 mm -> 11 x 6.7 mm
- board text removed: "+"
- board text removed: "-"
